File: AirQualityMonitor-SensorBoard.kicad_sch (KiCad schematic)
At the start: 3 parts

Commit message: Update page sizes
Connections:
- net VDD renamed VBUS
Changed lines of the file:
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@@
 	(generator "eeschema")
 	(generator_version "10.0")
-	(paper "A4")
+	(paper "A5" portrait)
 	(junction
 		(at 68.58 81.28)
@@
 		)
 	)
-	(label "VDD"
+	(label "VBUS"
 		(at 88.9 63.5 180)
 		(effects
@@
 		)
 	)
-	(label "VDD"
+	(label "VBUS"
 		(at 82.55 124.46 90)
 		(effects
